File: hardware/what-the-frequency-mk-5.brd (EAGLE design)
At the start: 77 x 44.5 mm, 37 parts, among them IC1 4040N, J1 POWER_JACKPTH, J2 AVR_ISP, U1 ATMEGA328P, U2 LCD-16X28X2, Y1 16MHz

Commit message: blah
Parts:
- removed R3: ???, A_butts:RESISTOR-AXIAL-PTH-5.08MM
- removed U$1: (no value), A_butts:COW_SMALL
- CONTRAST: value (none) -> 10k
- moved U$3 14.2 mm to (66.9, 3.07)
- moved U$7 14.1 mm to (63.7, 3.11)
- moved U$4 12.4 mm to (74.5, 15.2)
- moved U$2 12.4 mm to (74.6, 15.2)
- moved JP1 7.64 mm to (65.1, 11.0), turned to 270 degrees
Connections:
- removed net N$10: JP1.3, R3.P$1
- net GND: now also JP1.2; no longer JP1.1
- net VCC: now also JP1.1; no longer R3.P$2
- net XOUT: now also JP1.3; no longer JP1.2
Routing:
- net GND: track 67.4 -> 3.67 mm, vias 15 -> 0
- net VCC: track 169.3 -> 177.8 mm
- net N$10: track 5.88 -> 0.00 mm
Other:
- outline, holes or cut-outs redrawn
