File: hardware/crystal-test-breakout-mk-2.sch (EAGLE design)
At the start: 11 parts, among them Q1 1N3904

Commit message: klasdjcvkilasdjfl
Parts:
- C2: device A_butts:CAPACITOR-TRIM3050.504 -> A_butts:CAPACITOR-TRIM3040.427
- R2: device A_butts:POTENTIOMETER3296W-SIDE -> A_butts:POTENTIOMETER3296W
- Y1: device A_butts:RESONATORPTH -> A_butts:RESONATORPTH-BIGHOLES
Changed lines of the file:
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@@
 <?xml version="1.0" encoding="utf-8"?>
 <!DOCTYPE eagle SYSTEM "eagle.dtd">
-<eagle version="6.4">
+<eagle version="6.5.0">
 <drawing>
 <settings>
@@
 <setting verticaltext="up"/>
 </settings>
-<grid distance="100" unitdist="mil" unit="mil" style="lines" multiple="1" display="yes" altdistance="1" altunitdist="mm" altunit="mm"/>
+<grid distance="100" unitdist="mil" unit="mil" style="lines" multiple="1" display="yes" altdistance="1" altunitdist="mil" altunit="mil"/>
 <layers>
 <layer number="1" name="Top" color="4" fill="1" visible="yes" active="no"/>
@@
 <parts>
 <part name="JP1" library="A_butts" deviceset="M03" device="PTH"/>
-<part name="Y1" library="A_butts" deviceset="RESONATOR" device="PTH"/>
+<part name="Y1" library="A_butts" deviceset="RESONATOR" device="PTH-BIGHOLES"/>
 <part name="C1" library="A_butts" deviceset="CAPACITOR-CERAMIC" device="025-025X050"/>
 <part name="R1" library="A_butts" deviceset="RESISTOR" device="PTH-AXIAL-5.08MM"/>
 <part name="Q1" library="A_butts" deviceset="TRANSISTOR_NPN" device="TO-92-AMMO-EBC" value="1N3904"/>
-<part name="C2" library="A_butts" deviceset="CAPACITOR-TRIM" device="3050.504"/>
-<part name="R2" library="A_butts" deviceset="POTENTIOMETER" device="3296W-SIDE"/>
+<part name="C2" library="A_butts" deviceset="CAPACITOR-TRIM" device="3040.427"/>
+<part name="R2" library="A_butts" deviceset="POTENTIOMETER" device="3296W"/>
 <part name="GND1" library="A_butts" deviceset="GND" device=""/>
 <part name="SUPPLY1" library="A_butts" deviceset="VCC" device=""/>
@@
 <junction x="55.88" y="58.42"/>
 <pinref part="R2" gate="G$1" pin="E"/>
-<wire x1="53.34" y1="73.66" x2="55.88" y2="73.66" width="0.1524" layer="91"/>
+<wire x1="48.26" y1="78.74" x2="55.88" y2="73.66" width="0.1524" layer="91"/>
 <junction x="55.88" y="73.66"/>
 </segment>
@@
 <junction x="71.12" y="58.42"/>
 <pinref part="R2" gate="G$1" pin="S"/>
-<wire x1="48.26" y1="78.74" x2="48.26" y2="81.28" width="0.1524" layer="91"/>
+<wire x1="43.18" y1="73.66" x2="48.26" y2="81.28" width="0.1524" layer="91"/>
 <wire x1="71.12" y1="58.42" x2="76.2" y2="58.42" width="0.1524" layer="91"/>
 <wire x1="76.2" y1="58.42" x2="76.2" y2="55.88" width="0.1524" layer="91"/>
